File: air.brd (EAGLE design)
At the start: 100 x 80 mm, 32 parts, among them Q1 FC-12M, Q2 FC-26M, U1 ESP8266, U2 W25Q32FV, U3 CH340G, U4 AMS1117-3.3

Commit message: Add capeboard schematic and led on main schematic
Connections:
- net N$13 renamed PWM_GREEN
- new net PWM_BLUE: U1.9
- new net PWM_RED: U1.10
Changed lines of the file:
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@@
 <wire x1="-33.54" y1="17.82" x2="-56.83" y2="-24.13" width="0" layer="19" extent="1-1"/>
 </signal>
-<signal name="N$13">
+<signal name="PWM_GREEN">
 <contactref element="U1" pad="13"/>
 <contactref element="R5" pad="2"/>
@@
 <wire x1="-32.54" y1="17.82" x2="-18.78" y2="33.74" width="0" layer="19" extent="1-1"/>
 </signal>
+<signal name="PWM_RED">
+<contactref element="U1" pad="10"/>
+</signal>
+<signal name="PWM_BLUE">
+<contactref element="U1" pad="9"/>
+</signal>
 </signals>
